Commit message: added the the meshes tho the bot and the wheels are moving fine. No movement in Rviz as there is no odom frame however the wheels are moving fine. current engine ubeing used is DART only. In gaze bo no solid moment

File: src/bot/description/gazebo_controller.xacro (robot description, xacro)
@@ -9,15 +9,23 @@
             <back_left_joint>back_left_joint</back_left_joint>
             <back_right_joint>back_right_joint</back_right_joint>
-            <wheel_separation>0.34</wheel_separation> <wheelbase>0.4</wheelbase>
+            <!-- Updated to match actual mesh radius: 0.0323 m -->
+            <wheel_radius>0.0323</wheel_radius>
             <!--
-                wheelbase is the distance between front and rear wheel centres:
-                  chassis_length/2 - wheel_radius = 0.25 - 0.05 = 0.20 per side
-                  total = 0.40  (this was already correct)
+                wheel_separation = chassis_width/2 + wheel_thickness/2 (per side) x2
+                = 0.15 + (0.0352/2) = 0.15 + 0.0176 = 0.1676 per side
+                total = 0.3352
             -->
-            <wheel_radius>0.05</wheel_radius>
+            <wheel_separation>0.3352</wheel_separation>
+            <!--
+                wheelbase = (chassis_length/2 - wheel_radius) (per side) x2
+                = 0.25 - 0.0323 = 0.2177 per side
+                total = 0.4354
+            -->
+            <wheelbase>0.4354</wheelbase>
+            <!-- Required: without this the plugin ignores /cmd_vel from the bridge -->
+            <topic>/cmd_vel</topic>
             <publish_odom>true</publish_odom>
             <publish_odom_tf>true</publish_odom_tf>
             <publish_wheel_tf>true</publish_wheel_tf>
-            <topic>/cmd_vel</topic>
             <odom_topic>/odom</odom_topic>
             <tf_topic>/tf</tf_topic>
@@ -29,5 +37,6 @@
             filename="ignition-gazebo-joint-state-publisher-system"
             name="ignition::gazebo::systems::JointStatePublisher">
-            <topic>/joint_states</topic> <joint_name>front_left_joint</joint_name>
+            <topic>/joint_states</topic>
+            <joint_name>front_left_joint</joint_name>
             <joint_name>front_right_joint</joint_name>
             <joint_name>back_left_joint</joint_name>

File: src/bot/description/robot.urdf.xacro (robot description, xacro)
@@ -3,13 +3,20 @@
     <xacro:include filename="bot_core.xacro" />
     <xacro:include filename="wheel.xacro" />
-        <!--
-        BUG FIX 1: The file on disk is gazebo_controller.xacro, not
-        gazebo_control.xacro. Xacro will throw a FileNotFoundError (or
-        silently produce an incomplete URDF) with the wrong name.
-    -->
     <xacro:include filename="gazebo_controller.xacro" />
-    <xacro:mecanum_wheel prefix="front_left" x_reflect="1" y_reflect="1" />
-    <xacro:mecanum_wheel prefix="front_right" x_reflect="1" y_reflect="-1" />
-    <xacro:mecanum_wheel prefix="back_left" x_reflect="-1" y_reflect="1" />
-    <xacro:mecanum_wheel prefix="back_right" x_reflect="-1" y_reflect="-1" />
+    <xacro:mecanum_wheel
+        prefix="front_left"
+        x_reflect="1"  y_reflect="1"
+        mesh_file="front_left_wheel_X3.STL"/>
+    <xacro:mecanum_wheel
+        prefix="front_right"
+        x_reflect="1"  y_reflect="-1"
+        mesh_file="front_left_wheel_X3.STL"/>
+    <xacro:mecanum_wheel
+        prefix="back_left"
+        x_reflect="-1" y_reflect="1"
+        mesh_file="back_left_wheel_X3.STL"/>
+    <xacro:mecanum_wheel
+        prefix="back_right"
+        x_reflect="-1" y_reflect="-1"
+        mesh_file="back_left_wheel_X3.STL"/>
 </robot>

File: src/bot/description/wheel.xacro (robot description, xacro)
@@ -1,20 +1,85 @@
 <?xml version="1.0"?>
 <robot xmlns:xacro="http://www.ros.org/wiki/xacro">
-    <xacro:property name="wheel_radius" value="0.05"/>
-    <xacro:property name="wheel_thickness" value="0.04"/>
-    <xacro:macro name="mecanum_wheel" params="prefix x_reflect y_reflect">
+    <!--
+        Dimensions measured directly from the STL bounding boxes (units: meters).
+        Do NOT change these back to 0.05/0.04 — those were guesses and are wrong.
+        wheel_radius    = 0.0323  (half of X/Y span of mesh)
+        wheel_thickness = 0.0352  (Z span of mesh)
+        mesh_z_offset   = 0.0024  (mesh was exported with centroid slightly off-origin;
+                                   negating this in the visual origin re-centers it)
+    -->
+    <xacro:property name="wheel_radius"    value="0.0323"/>
+    <xacro:property name="wheel_thickness" value="0.0352"/>
+    <xacro:property name="mesh_z_offset"   value="0.0024"/>
+    <xacro:property name="mesh_pkg" value="file://$(find bot)/meshes"/>
+    <!--
+        mecanum_wheel macro
+        params:
+          prefix     — joint/link name prefix (front_left, front_right, …)
+          x_reflect  — +1 front, -1 rear
+          y_reflect  — +1 left,  -1 right
+          mesh_file  — STL filename (without path), e.g. front_left_wheel_X3.STL
+        Right-side wheels are the mirror image of left-side wheels.
+        We achieve this by scaling the mesh by (1, -1, 1) in Y, which flips the
+        roller angle from one diagonal to the other — exactly the physical
+        difference between left and right mecanum wheels. The collision geometry
+        stays a plain cylinder regardless of side (the MecanumDrive plugin handles
+        kinematics; we don't need physically-accurate roller contacts here).-->
+    <xacro:macro name="mecanum_wheel" params="prefix x_reflect y_reflect mesh_file">
         <joint name="${prefix}_joint" type="continuous">
             <parent link="chassis"/>
-            <child link="${prefix}_wheel"/>
-            <origin xyz="${x_reflect*(chassis_length/2 - wheel_radius)} ${y_reflect*(chassis_width/2 + wheel_thickness/2)} -0.05" rpy="${pi/2} 0 0"/>
+            <child  link="${prefix}_wheel"/>
+            <!--
+                Joint X: place wheel near the chassis corner.
+                         chassis_length/2 - wheel_radius keeps the wheel edge
+                         flush with the chassis end rather than sticking out.
+                Joint Y: move outward by half chassis width + half wheel thickness
+                         so the wheel face sits just outside the chassis body.
+                Joint Z: -0.05 drops the wheel below the chassis centre so it
+                         sits on the ground (chassis is raised 0.1 m by chassis_joint).
+                RPY pi/2 around X: rotates the child frame so the wheel's Z axis
+                         (its spin axis in the mesh) aligns with the world Y axis,
+                         i.e. the wheel rolls fore/aft as expected.
+            -->
+            <origin
+                xyz="${x_reflect * (chassis_length/2 - wheel_radius)}
+                     ${y_reflect * (chassis_width/2  + wheel_thickness/2)}
+                     -0.05"
+                rpy="${pi/2} 0 0"/>
             <axis xyz="0 0 -1"/>
         </joint>
         <link name="${prefix}_wheel">
+            <!-- ── VISUAL: actual mecanum mesh ──────────────────────────────── -->
             <visual>
+                <origin xyz="0 0 ${-mesh_z_offset}" rpy="0 0 0"/>
+                <!--
+                    mesh_z_offset correction: the STL centroid sits 0.0024 m above
+                    the mesh geometric centre. Shifting by -mesh_z_offset in the
+                    visual origin pulls it back to the joint centre so the wheel
+                    doesn't appear to float or sink relative to the joint frame.
+                -->
                 <geometry>
-                    <cylinder radius="${wheel_radius}" length="${wheel_thickness}"/>
+                    <mesh
+                        filename="${mesh_pkg}/${mesh_file}"
+                        scale="1 ${y_reflect} 1"/>
+                    <!--
+                        scale Y by y_reflect:
+                          left  wheels (y_reflect= 1) → scale  1  1  1 → mesh as-is
+                          right wheels (y_reflect=-1) → scale  1 -1  1 → mirrored in Y,
+                          which flips the roller diagonal from \ to /
+                    -->
                 </geometry>
-                <material name="black"><color rgba="0.1 0.1 0.1 1"/></material>
             </visual>
+            <!-- ── COLLISION: simple cylinder ───────────────────────────────── -->
+            <!--
+                Using a cylinder (not the mesh) for collision because:
+                  1. The MecanumDrive plugin computes holonomic kinematics algebraically;
+                     it does not depend on contact geometry.
+                  2. Cylinder collision is stable and fast. Mesh collision with
+                     44 k triangles and free-spinning roller sub-geometry causes
+                     numerical instability in DART's contact solver.
+                  3. The cylinder dimensions match the mesh bounding circle so
+                     ground clearance and chassis clearance are still correct.
+            -->
             <collision>
                 <geometry>
@@ -22,5 +87,9 @@
                 </geometry>
             </collision>
-            <xacro:inertial_cylinder mass="0.2" length="${wheel_thickness}" radius="${wheel_radius}">
+            <!-- ── INERTIA: solid cylinder approximation ────────────────────── -->
+            <xacro:inertial_cylinder
+                mass="0.2"
+                length="${wheel_thickness}"
+                radius="${wheel_radius}">
                 <origin xyz="0 0 0" rpy="0 0 0"/>
             </xacro:inertial_cylinder>
